Commit message: better dimensions / position in example

File: objects/urdf/bluerov.xacro (robot description, xacro)
@@ -2,13 +2,9 @@
 <robot name="bluerov" xmlns:xacro="http://www.ros.org/wiki/xacro">
 <xacro:arg name="prefix" default="bluerov"/>
-    <material name="brovgrey">
-    <color rgba="0.25 0.25 0.28 1"/>
-  </material>
-  <link name="$(arg prefix)/base_link">
+<link name="$(arg prefix)/base_link">
     <visual>
       <geometry>
         <mesh filename="package://marine_presenter/objects/mesh/bluerov2_noprop.ive"/>
       </geometry>
-      <material name="brovgrey"/>
     </visual>
   </link>
